Commit message: Fully completed package, final commit of my custom gym environment :D

File: pybullet_workshop_23/envs/urdf/arena/track.urdf (robot description, URDF)
Before this commit: robot cube, 2 links, 1 joints
Links:
- link base_link: mass 1000.0 -> 1000000.0
- link path: mass 1000.0 -> 1000000.0
